Commit message: v3.2

File: arm_20/robotic_arm_20/robots/robotic_arm_20.urdf (robot description, URDF)
Before this commit: robot robotic_arm_20, 8 links, 7 joints
Links:
- added link camera, mass 0.1; collision box size=0.05 0.05 0.05; visual box size=0.05 0.05 0.05
Joints:
- added joint camera_joint: type fixed, parent link_3, child camera, origin xyz=0.4 0 0.2 rpy=0 0 0, axis 1 1 0

File: arm_20/robotic_arm_20/urdf/robotic_arm_20.urdf (robot description, URDF)
Before this commit: robot robotic_arm_20, 8 links, 7 joints
Links:
- added link camera, mass 0.1; collision box size=0.05 0.05 0.05; visual box size=0.005 0.005 0.005
Joints:
- added joint camera_joint: type fixed, parent link_4, child camera, origin xyz=0.4 0 0.2 rpy=1.57 0 0, axis 1 1 0
- joint joint_1: limit lower=-3.14 upper=3.14 effort=100 velocity=20 -> lower=-3.14 upper=3.14 effort=200 velocity=20
- joint joint_2: limit lower=-3.14 upper=3.14 effort=100 velocity=20 -> lower=-3.14 upper=3.14 effort=200 velocity=20
- joint joint_3: limit lower=-3.14 upper=3.14 effort=100 velocity=20 -> lower=-3.14 upper=3.14 effort=200 velocity=20
- joint joint_4: limit lower=-3.14 upper=3.14 effort=100 velocity=20 -> lower=-3.14 upper=3.14 effort=200 velocity=20
- joint joint_5: limit lower=-3.14 upper=3.14 effort=100 velocity=20 -> lower=-3.14 upper=3.14 effort=200 velocity=20
- joint joint_6: limit lower=-3.14 upper=3.14 effort=100 velocity=20 -> lower=-3.14 upper=3.14 effort=200 velocity=20
